File: EAGLE/Theremizer.sch (EAGLE design)
At the start: 166 parts, among them IC1 AS3320, IC2 NE5532N, IC3 TL072D, IC4 NE5532N, J1 3x2 M, J2 1x6 M, J3 AUDIO_JACK_TRS_0.25"_PTH_RA, J4 POWER_JACK, J5 AUDIO_JACK_TRS_0.25"_PTH_RA, Q1 PMV45EN2R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

Commit message: Redid layout, hopefully better
Parts:
- removed R49: 0, rcl:R-US_R0805
- removed TP2: TPPAD1-13, testpad:TPPAD1-13
- added JP10, JP11, JP12: (no value), jumper:JP1E
- R20, R8: value 0 -> 15k; MPN RC0805JR-070RL -> RC0805FR-0710KL
- R34: device pot:TRIM_US-PT10 -> pot:TRIM_US-B64Y
Connections:
- new net N$75: C40.2, C41.2, U5.OUTA
- new net N$77: R43.E, R8.1
- new net N$78: R20.1, R44.E
- net +15V: now also JP10.2; no longer R20.2
- net +5V: now also JP12.2, R20.2, R8.2; no longer R43.E, R44.E, R8.1
- net -15V: now also JP11.1; no longer R49.2
- net 5VEXT: now also JP12.1; no longer R8.2, TP2.TP
- net N$55: now also JP10.1; no longer R20.1
- net N$56: now also JP11.2; no longer R49.1
- net THEREMIN_OUT: no longer C40.2, C41.2, U5.OUTA
Other:
- moved on the sheet: R20, R43, R44, R8

Commit message: Board laid out by hand, still needs vias
Parts:
- C32: value 10u -> 0.1u
Connections:
- removed net N$47: J5.EARTH-NORM
- net GND: now also J5.EARTH-NORM, U4.INC, U4.IND
Changed lines of the file:
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@@
 <clearance class="0" value="0.1524"/>
 </class>
-<class number="1" name="power" width="0.4064" drill="0">
+<class number="1" name="power" width="1" drill="0">
 </class>
 <class number="4" name="test" width="0" drill="0">
@@
 <part name="C30" library="rcl" library_urn="urn:adsk.eagle:library:334" deviceset="C-EU" device="C0805" package3d_urn="urn:adsk.eagle:package:23617/2" value="2.2n"/>
 <part name="C31" library="rcl" library_urn="urn:adsk.eagle:library:334" deviceset="C-EU" device="C0805" package3d_urn="urn:adsk.eagle:package:23617/2" value="470p"/>
-<part name="C32" library="rcl" library_urn="urn:adsk.eagle:library:334" deviceset="C-EU" device="C0805" package3d_urn="urn:adsk.eagle:package:23617/2" value="10u"/>
+<part name="C32" library="rcl" library_urn="urn:adsk.eagle:library:334" deviceset="C-EU" device="C0805" package3d_urn="urn:adsk.eagle:package:23617/2" value="0.1u"/>
 <part name="R34" library="pot" library_urn="urn:adsk.eagle:library:331" deviceset="TRIM_US-" device="B64Y" package3d_urn="urn:adsk.eagle:package:22690/1" value="22k"/>
 <part name="R25" library="rcl" library_urn="urn:adsk.eagle:library:334" deviceset="R-US_" device="R0805" package3d_urn="urn:adsk.eagle:package:23553/2" value="100k"/>
@@
 <attribute name="MPN" value="RC0805FR-0710KL"/>
 </part>
+<part name="GND25" library="supply1" library_urn="urn:adsk.eagle:library:371" deviceset="GND" device=""/>
 </parts>
 <sheets>
@@
 <pinref part="U4" gate="A" pin="REFSEL"/>
 <wire x1="166.37" y1="93.98" x2="167.64" y2="93.98" width="0.1524" layer="91"/>
-<wire x1="151.13" y1="93.98" x2="165.1" y2="93.98" width="0.1524" layer="91"/>
+<wire x1="151.13" y1="93.98" x2="156.21" y2="93.98" width="0.1524" layer="91"/>
+<pinref part="U4" gate="A" pin="INC"/>
+<wire x1="156.21" y1="93.98" x2="161.29" y2="93.98" width="0.1524" layer="91"/>
+<wire x1="161.29" y1="93.98" x2="165.1" y2="93.98" width="0.1524" layer="91"/>
+<wire x1="151.13" y1="88.9" x2="156.21" y2="88.9" width="0.1524" layer="91"/>
+<wire x1="156.21" y1="88.9" x2="156.21" y2="93.98" width="0.1524" layer="91"/>
+<junction x="156.21" y="93.98"/>
+<pinref part="U4" gate="A" pin="IND"/>
+<wire x1="151.13" y1="86.36" x2="161.29" y2="86.36" width="0.1524" layer="91"/>
+<wire x1="161.29" y1="86.36" x2="161.29" y2="93.98" width="0.1524" layer="91"/>
+<junction x="161.29" y="93.98"/>
 </segment>
 <segment>
@@
 </segment>
 </net>
-<net name="VIN" class="0">
+<net name="VIN" class="1">
 <segment>
 <wire x1="308.61" y1="213.36" x2="298.45" y2="213.36" width="0.1524" layer="91"/>
@@
 </segment>
 </net>
-<net name="N$3" class="0">
+<net name="N$3" class="1">
 <segment>
 <pinref part="D2" gate="G$1" pin="A"/>
@@
 </segment>
 </net>
-<net name="5VEXT" class="0">
+<net name="5VEXT" class="1">
 <segment>
 <wire x1="326.39" y1="213.36" x2="336.55" y2="213.36" width="0.1524" layer="91"/>
@@
 </segment>
 </net>
-<net name="N$51" class="0">
+<net name="N$51" class="1">
 <segment>
 <pinref part="J4" gate="G$1" pin="PWR"/>
@@
 </segment>
 </net>
-<net name="N$54" class="0">
+<net name="N$54" class="1">
 <segment>
 <pinref part="D4" gate="G$1" pin="C"/>
@@
 </segment>
 </net>
-<net name="N$55" class="0">
+<net name="N$55" class="1">
 <segment>
 <pinref part="U3" gate="G$1" pin="+VOUT"/>
@@
 </segment>
 </net>
-<net name="N$56" class="0">
+<net name="N$56" class="1">
 <segment>
 <pinref part="JP11" gate="A" pin="2"/>
@@
 </segment>
 </net>
-<net name="N$77" class="1">
+<net name="N$77" class="0">
 <segment>
 <pinref part="R43" gate="G$1" pin="E"/>
@@
 </segment>
 </net>
-<net name="N$78" class="1">
+<net name="N$78" class="0">
 <segment>
 <pinref part="R44" gate="G$1" pin="E"/>
@@
 <junction x="93.98" y="124.46"/>
 <pinref part="IC1" gate="G$1" pin="3"/>
-<wire x1="124.46" y1="132.08" x2="106.68" y2="132.08" width="0.1524" layer="91"/>
-<wire x1="124.46" y1="132.08" x2="93.98" y2="132.08" width="0.1524" layer="91"/>
+<wire x1="124.46" y1="132.08" x2="114.3" y2="132.08" width="0.1524" layer="91"/>
+<wire x1="114.3" y1="132.08" x2="106.68" y2="132.08" width="0.1524" layer="91"/>
+<wire x1="124.46" y1="132.08" x2="114.3" y2="132.08" width="0.1524" layer="91"/>
 <pinref part="C10" gate="G$1" pin="1"/>
+<wire x1="114.3" y1="132.08" x2="93.98" y2="132.08" width="0.1524" layer="91"/>
 <wire x1="96.52" y1="129.54" x2="93.98" y2="129.54" width="0.1524" layer="91"/>
 <junction x="93.98" y="129.54"/>
+<wire x1="124.46" y1="132.08" x2="114.3" y2="132.08" width="0.1524" layer="91"/>
+<junction x="124.46" y="132.08"/>
+<junction x="114.3" y="132.08"/>
 </segment>
 <segment>
@@
 <attribute name="VALUE" x="53.34" y="71.882" size="1.778" layer="96" rot="R180"/>
 </instance>
-<instance part="GND23" gate="1" x="55.88" y="67.31" smashed="yes">
-<attribute name="VALUE" x="53.34" y="64.77" size="1.778" layer="96"/>
+<instance part="GND23" gate="1" x="55.88" y="64.77" smashed="yes">
+<attribute name="VALUE" x="53.34" y="62.23" size="1.778" layer="96"/>
 </instance>
 <instance part="C11" gate="G$1" x="63.5" y="92.71" smashed="yes">
@@
 <attribute name="VALUE" x="261.62" y="44.958" size="1.778" layer="96"/>
 </instance>
+<instance part="GND25" gate="1" x="232.41" y="87.63" smashed="yes">
+<attribute name="VALUE" x="229.87" y="85.09" size="1.778" layer="96"/>
+</instance>
 </instances>
 <busses>
@@
 <pinref part="R30" gate="G$1" pin="1"/>
 <pinref part="GND23" gate="1" pin="GND"/>
-<wire x1="55.88" y1="68.58" x2="55.88" y2="69.85" width="0.1524" layer="91"/>
+<wire x1="55.88" y1="67.31" x2="55.88" y2="69.85" width="0.1524" layer="91"/>
 </segment>
 <segment>
@@
 </segment>
 <segment>
-<pinref part="C26" gate="G$1" pin="2"/>
-<wire x1="29.21" y1="161.29" x2="29.21" y2="151.13" width="0.1524" layer="91"/>
-<pinref part="GND31" gate="1" pin="GND"/>
-<pinref part="Q3" gate="1" pin="G"/>
-<wire x1="29.21" y1="151.13" x2="29.21" y2="129.54" width="0.1524" layer="91"/>
-<wire x1="31.75" y1="151.13" x2="29.21" y2="151.13" width="0.1524" layer="91"/>
-<junction x="29.21" y="151.13"/>
-</segment>
-<segment>
 <wire x1="20.32" y1="45.72" x2="20.32" y2="55.88" width="0.1524" layer="91"/>
 <pinref part="GND20" gate="1" pin="GND"/>
@@
 <wire x1="271.78" y1="48.26" x2="270.51" y2="48.26" width="0.1524" layer="91"/>
 </segment>
+<segment>
+<pinref part="C26" gate="G$1" pin="2"/>
+<wire x1="29.21" y1="161.29" x2="29.21" y2="151.13" width="0.1524" layer="91"/>
+<pinref part="Q3" gate="1" pin="G"/>
+<wire x1="31.75" y1="151.13" x2="29.21" y2="151.13" width="0.1524" layer="91"/>
+<pinref part="GND31" gate="1" pin="GND"/>
+<wire x1="29.21" y1="129.54" x2="31.75" y2="129.54" width="0.1524" layer="91"/>
+<wire x1="31.75" y1="129.54" x2="31.75" y2="151.13" width="0.1524" layer="91"/>
+<junction x="31.75" y="151.13"/>
+</segment>
+<segment>
+<pinref part="J5" gate="G$1" pin="EARTH-NORM"/>
+<wire x1="229.87" y1="92.71" x2="232.41" y2="92.71" width="0.1524" layer="91"/>
+<pinref part="GND25" gate="1" pin="GND"/>
+<wire x1="232.41" y1="90.17" x2="232.41" y2="92.71" width="0.1524" layer="91"/>
+</segment>
 </net>
 <net name="N$1" class="0">
@@
 </segment>
 </net>
-<net name="N$47" class="0">
-<segment>
-<pinref part="J5" gate="G$1" pin="EARTH-NORM"/>
-<wire x1="229.87" y1="92.71" x2="232.41" y2="92.71" width="0.1524" layer="91"/>
-</segment>
-</net>
 <net name="OUTPUT" class="0">
 <segment>
@@
 </segment>
 </net>
-<net name="N$68" class="0">
-<segment>
-<junction x="29.21" y="151.13"/>
-</segment>
-</net>

Commit message: Final Schematic/Board Layout
Parts:
- added D5: M7, diode:MBRA340T3
- D1: device diode:DIODE-SMB -> diode:MBRA340T3
- D4: value M7 -> MBRA340T3; device diode:DIODE-SMB -> diode:MBRA340T3; MFR SMC Diode -> (none); MPN 10BQ030TR -> (none)
- R36, R37, R43, R44, R45, R47, R57, R59: device pot:TRIM_US-ECP10P -> pot:TRIM_US-B64Y
Connections:
- new net N$47: C50.1, D5.C, U6.IN
- net N$51: now also D5.A; no longer C50.1, U6.IN
Other:
- moved on the sheet: R59
